File: Eagle/Sheamtic.brd (EAGLE design)
At the start: 100 x 80 mm, 21 parts, among them IC1 PIC16F874P

Commit message: board
Parts:
- moved R4 165.4 mm to (95.2, 35.6), turned to 90 degrees
- moved JP1 156.7 mm to (91.4, 76.2), turned to 180 degrees
- moved R3 154.2 mm to (90.2, 22.9), turned to 90 degrees
- moved R2 150.6 mm to (96.5, 22.9), turned to 90 degrees
- moved LED1 138.6 mm to (95.2, 57.1), turned to 90 degrees
- moved LED2 138.6 mm to (82.5, 57.1), turned to 90 degrees
- moved R1 119.9 mm to (73.7, 22.9), turned to 270 degrees
- moved R6 116.5 mm to (81.3, 36.8), turned to 90 degrees
- moved R5 113.0 mm to (87.6, 36.8), turned to 270 degrees
- moved C3 111.9 mm to (81.3, 48.3), turned to 90 degrees
- moved S1 111.7 mm to (77.5, 6.35)
- moved C2 100.8 mm to (64.8, 20.3), turned to 180 degrees
- moved Q1 100.5 mm to (71.1, 71.1), turned to 270 degrees
- moved DIS2 96.5 mm to (30.5, 12.7)
- moved IC1 95.2 mm to (54.6, 50.8), turned to 90 degrees
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Routing:
- net GND: track 0.00 -> 464.8 mm
- net VCC: track 0.00 -> 210.1 mm
- net N$34: track 0.00 -> 183.9 mm
- net N$23: track 0.00 -> 76.4 mm
- net N$35: track 0.00 -> 76.3 mm
- net N$2: track 0.00 -> 63.2 mm
- net N$1: track 0.00 -> 62.4 mm
- net N$19: track 0.00 -> 62.0 mm
- net N$18: track 0.00 -> 61.0 mm
- net N$15: track 0.00 -> 58.6 mm
- net N$14: track 0.00 -> 55.5 mm
- net N$13: track 0.00 -> 53.0 mm
- net N$11: track 0.00 -> 49.3 mm
- net N$7: track 0.00 -> 41.6 mm
- net N$26: track 0.00 -> 40.0 mm
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
Commit message: update board
Parts:
- moved IC2 26.7 mm to (11.4, 52.1), turned to 180 degrees
- moved C1 22.7 mm to (90.2, 45.7)
- moved R1 17.3 mm to (83.8, 36.8)
- moved IC3 16.9 mm to (30.5, 38.1), turned to 180 degrees
- moved C2 12.7 mm to (64.8, 7.62), turned to 90 degrees
- moved R6 11.4 mm to (69.8, 36.8)
- moved X1 6.48 mm to (48.3, 12.7)
- moved JP1 5.68 mm to (96.5, 73.7), turned to 90 degrees
- moved C3 5.68 mm to (76.2, 45.7), turned to 270 degrees
- moved DIS2 5.39 mm to (26.7, 16.5)
- moved DIS1 3.81 mm to (12.7, 16.5)
- moved R3 3.81 mm to (86.4, 22.9)
- moved LED2 2.54 mm to (85.1, 57.1)
- moved R5 2.54 mm to (90.2, 36.8)
- moved R2 2.54 mm to (94.0, 22.9)
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Routing:
- net N$34: track 183.9 -> 0.00 mm
- net GND: track 464.8 -> 364.9 mm
- net N$8: track 0.00 -> 67.9 mm
- net N$23: track 76.4 -> 25.7 mm
- net N$22: track 0.00 -> 50.1 mm
- net VCC: track 210.1 -> 250.9 mm
- net N$14: track 55.5 -> 15.3 mm
- net N$15: track 58.6 -> 18.6 mm
- net N$13: track 53.0 -> 13.0 mm
- net N$21: track 0.00 -> 39.9 mm
- net N$20: track 0.00 -> 39.9 mm
- net N$32: track 0.00 -> 39.8 mm
- net N$5: track 22.3 -> 62.1 mm
- net N$9: track 19.9 -> 59.6 mm
- net N$11: track 49.3 -> 9.94 mm
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
Commit message: Eagle
Routing:
- net N$34: track 0.00 -> 34.1 mm, vias 0 -> 2
- net N$33: track 0.00 -> 9.20 mm, vias 0 -> 2
- net N$5: track 62.1 -> 66.6 mm
- net VCC: track 250.9 -> 253.1 mm
- added copper zone on layer 16, net GND
Other:
- board text added: "Groupe 3"
Changed lines of the file:
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@@
 <wire x1="100" y1="80" x2="0" y2="80" width="0" layer="20"/>
 <wire x1="0" y1="80" x2="0" y2="0" width="0" layer="20"/>
+<text x="86.36" y="3.81" size="1.778" layer="1">Groupe 3</text>
 </plain>
 <attributes>
@@
 <wire x1="50.8" y1="46.99" x2="50.8" y2="12.7" width="0.381" layer="16"/>
 <wire x1="50.8" y1="12.7" x2="50.7746" y2="12.7" width="0.381" layer="16"/>
-<wire x1="13.6525" y1="60.6425" x2="8.89" y2="55.88" width="0.381" layer="16"/>
-<wire x1="28.8925" y1="60.6425" x2="13.6525" y2="60.6425" width="0.381" layer="16"/>
+<wire x1="9.8425" y1="60.6425" x2="8.89" y2="59.69" width="0.381" layer="16"/>
+<wire x1="8.89" y1="59.69" x2="8.89" y2="55.88" width="0.381" layer="16"/>
+<wire x1="28.8925" y1="60.6425" x2="9.8425" y2="60.6425" width="0.381" layer="16"/>
 <wire x1="42.545" y1="46.99" x2="28.8925" y2="60.6425" width="0.381" layer="16"/>
 <wire x1="46.99" y1="46.99" x2="42.545" y2="46.99" width="0.381" layer="16"/>
@@
 <wire x1="45.72" y1="12.7" x2="39.0525" y2="6.0325" width="0.381" layer="16"/>
 <wire x1="45.72" y1="12.7" x2="45.7708" y2="12.7" width="0.381" layer="16"/>
+<polygon width="0.4572" layer="16" isolate="0.02031875">
+<vertex x="0" y="80.01"/>
+<vertex x="99.06" y="80.01"/>
+<vertex x="99.06" y="0"/>
+<vertex x="0" y="0"/>
+</polygon>
 </signal>
 <signal name="N$2">
@@
 <wire x1="60.325" y1="47.625" x2="60.325" y2="43.815" width="0.381" layer="16"/>
 <wire x1="60.96" y1="48.26" x2="60.325" y2="47.625" width="0.381" layer="16"/>
-<wire x1="63.5" y1="48.26" x2="60.96" y2="48.26" width="0.381" layer="16"/>
-<wire x1="65.0875" y1="49.8475" x2="63.5" y2="48.26" width="0.381" layer="16"/>
-<wire x1="65.0875" y1="54.2925" x2="65.0875" y2="49.8475" width="0.381" layer="16"/>
-<wire x1="63.5" y1="55.88" x2="65.0875" y2="54.2925" width="0.381" layer="16"/>
+<wire x1="67.6275" y1="48.26" x2="60.96" y2="48.26" width="0.381" layer="16"/>
+<wire x1="67.6275" y1="51.7525" x2="67.6275" y2="48.26" width="0.381" layer="16"/>
+<wire x1="63.5" y1="55.88" x2="67.6275" y2="51.7525" width="0.381" layer="16"/>
 <wire x1="60.96" y1="55.88" x2="63.5" y2="55.88" width="0.381" layer="16"/>
 <wire x1="60.325" y1="56.515" x2="60.96" y2="55.88" width="0.381" layer="16"/>
@@
 <wire x1="13.97" y1="55.88" x2="16.8275" y2="58.7375" width="0.381" layer="16"/>
 </signal>
-<signal name="N$12">
-<contactref element="IC2" pad="4"/>
-<contactref element="IC1" pad="40"/>
-<wire x1="11.43" y1="55.88" x2="46.99" y2="26.67" width="0" layer="19" extent="1-1"/>
-</signal>
 <signal name="N$11">
 <contactref element="IC3" pad="1"/>
@@
 <contactref element="IC1" pad="10"/>
 <contactref element="DIS1" pad="5"/>
-<wire x1="17.78" y1="8.89" x2="62.23" y2="49.53" width="0" layer="19" extent="1-1"/>
+<via x="19.05" y="38.1" extent="1-16" drill="0.381" diameter="1.3"/>
+<wire x1="17.78" y1="8.89" x2="19.05" y2="10.16" width="0.1524" layer="16"/>
+<wire x1="19.05" y1="10.16" x2="19.05" y2="38.1" width="0.1524" layer="16"/>
+<via x="66.04" y="50.8" extent="1-16" drill="0.4572" diameter="1.3"/>
+<wire x1="62.23" y1="49.53" x2="64.77" y2="49.53" width="0.4572" layer="16"/>
+<wire x1="64.77" y1="49.53" x2="66.04" y2="50.8" width="0.4572" layer="16"/>
+<wire x1="19.05" y1="38.1" x2="62.23" y2="49.53" width="0" layer="19" extent="1-1"/>
+</signal>
+<signal name="N$33">
+<via x="41.91" y="22.86" extent="1-16" drill="0.4572" diameter="1.3"/>
+<contactref element="IC2" pad="4"/>
+<contactref element="IC1" pad="40"/>
+<wire x1="41.91" y1="22.86" x2="45.72" y2="26.67" width="0.4572" layer="16"/>
+<wire x1="45.72" y1="26.67" x2="46.99" y2="26.67" width="0.4572" layer="16"/>
+<via x="11.43" y="58.42" extent="1-16" drill="0.4572" diameter="1.3"/>
+<wire x1="11.43" y1="55.88" x2="11.43" y2="58.42" width="0.4572" layer="16"/>
+<wire x1="41.91" y1="22.86" x2="11.43" y2="55.88" width="0" layer="19" extent="1-1"/>
 </signal>
 </signals>
